Commit message: add ave arm backpack2

File: src/arm_v2_tradition_new/urdf/arm_v2_tradition_new.urdf (robot description, URDF)
Before this commit: robot arm_v2_tradition_new, 8 links, 7 joints
Joints:
- joint joint1: limit lower=-180 upper=180 effort=0 velocity=0 -> lower=0 upper=70 effort=0 velocity=0
- joint joint2: limit lower=-180 upper=180 effort=0 velocity=0 -> lower=0 upper=80 effort=0 velocity=0
- joint joint3: limit (none) -> lower=-150 upper=0 effort=0 velocity=0
- joint joint4: axis 0 0 1 -> 0 0 -1; limit (none) -> lower=0 upper=135 effort=0 velocity=0
- joint joint5: axis 0 0 1 -> 0 0 -1; limit (none) -> lower=0 upper=135 effort=0 velocity=0

File: src/ave_arm_backpack2/config/gazebo_arm_v2_tradition_new.urdf (robot description, URDF)
Before this commit: robot arm_v2_tradition_new, 9 links, 8 joints
Links:
- removed link world
Joints:
- removed joint fixed
- joint joint2: limit lower=-180 upper=180 effort=0 velocity=0 -> lower=0 upper=80 effort=0 velocity=0
- joint joint3: limit (none) -> lower=-150 upper=0 effort=0 velocity=0
- joint joint4: axis 0 0 1 -> 0 0 -1; limit (none) -> lower=0 upper=135 effort=0 velocity=0
- joint joint5: axis 0 0 1 -> 0 0 -1; limit (none) -> lower=0 upper=135 effort=0 velocity=0
